File: pcb/esp32-u4wdh.kicad_sch (KiCad schematic)
At the start: 9 parts, among them IC1 ESP32-U4WDH, SW1 SW_Push

Commit message: ADD 3D Models for all footprints, export new PCB Image and remove D1 for R8 with 0R (Jumper R)
Parts:
- removed A1: YAGEO_ANT3216LL00R2300A, RF_Antenna:YAGEO_ANT3216LL00R2300A, symbol RF_Antenna:YAGEO_ANT3216LL00R2300A
- added A1: YAGEO_ANT3216LL00R2400A, RF_Antenna:YAGEO_ANT3216LL00R2400A, symbol RF_Antenna:YAGEO_ANT3216LL00R2400A
Connections:
- net at C1.1, L1.1: now also A1.1 (Feed-In)
Changed lines of the file:
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@@
     (pin "1")
+  )
+  (symbol (lib_id "RF_Antenna:YAGEO_ANT3216LL00R2400A") (at 60.96 62.23 180) (unit 1)
+    (in_bom yes) (on_board yes) (fields_autoplaced)
+    (property "Reference" "A1" (id 0) (at 60.96 54.61 0))
+    (property "Value" "YAGEO_ANT3216LL00R2400A" (id 1) (at 60.96 57.15 0))
+    (property "Footprint" "RF_Antenna:YAGEO_ANT3216LL00R2400A" (id 2) (at 64.77 62.23 0)
+      (effects (font (size 1.27 1.27)) hide)
+    )
+    (property "Datasheet" "" (id 3) (at 64.77 62.23 0)
+      (effects (font (size 1.27 1.27)) hide)
+    )
+    (pin "1")
+    (pin "2")
   )
   (symbol (lib_id "power:+3.3VA") (at 93.98 114.3 0) (unit 1)
@@
     (pin "1")
   )
-  (symbol (lib_id "RF_Antenna:YAGEO_ANT3216LL00R2300A") (at 60.96 62.23 180) (unit 1)
-    (in_bom yes) (on_board yes) (fields_autoplaced)
-    (property "Reference" "A1" (id 0) (at 60.96 54.61 0))
-    (property "Value" "YAGEO_ANT3216LL00R2300A" (id 1) (at 60.96 57.15 0))
-    (property "Footprint" "RF_Antenna:YAGEO_ANT3216LL00R2300A" (id 2) (at 64.77 62.23 0)
-      (effects (font (size 1.27 1.27)) hide)
-    )
-    (property "Datasheet" "https://www.yageo.com/upload/media/product/productsearch/datasheet/wireless/An_Ceramiz_2450_3216_L00_0.pdf" (id 3) (at 64.77 62.23 0)
-      (effects (font (size 1.27 1.27)) hide)
-    )
-    (pin "1")
-    (pin "2")
-  )
   (symbol (lib_id "power:+3.3VA") (at 200.66 45.72 0) (unit 1)

Commit message: ADD new picture, and propper GND plane on top layer
Parts:
- C3: value 10uF -> 100nF
- R1: value 10K -> 100k
Changed lines of the file:
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@@
       (effects (font (size 1.27 1.27)) (justify left))
     )
-    (property "Value" "10uF" (id 1) (at 97.79 134.6199 0)
+    (property "Value" "100nF" (id 1) (at 97.79 134.6199 0)
       (effects (font (size 1.27 1.27)) (justify left))
     )
@@
       (effects (font (size 1.27 1.27)) (justify left))
     )
-    (property "Value" "10K" (id 1) (at 96.52 121.9199 0)
+    (property "Value" "100k" (id 1) (at 96.52 121.9199 0)
       (effects (font (size 1.27 1.27)) (justify left))
     )

Commit message: REF PCB Layout, Switch to new USB-C Receptable
Parts:
- C1: value 8pF -> 8p
- C2: value 10pF -> 10p
- C3: value 100nF -> 100n
- L1: value 1nH -> 1n
- R2: value 10K(5%) -> 100k
Connections:
- net ANTENNA: now also A1.1 (Feed-In), C1.1, L1.1
- net GPIO26: now reaches IC1.15 (GPIO26)
- net MTDI: now reaches IC1.18 (MTDI), R2.1
- net +3.3VA renamed +3V3
- net GPIO36: no longer names the net of IC1.5 (SENSOR_VP)
- no-connect marks 31 -> 32
Other:
- moved on the sheet: R2
